File: wch-link.kicad_sch (KiCad schematic)
At the start: 27 parts, among them J1 USB2.0_C_v3, P1 1Pin, U3 AMS1117-3.3, Y1 Oscillator_24GND

Commit message: v1
Parts:
- removed U2: ~, symbol $74th:WCH-Link-Header-L
- removed U4: ~, symbol $74th:WCH-Link-Header-R
- added C3, C4: 10u, $74th:Capacitor_0603_1608, symbol Device:C
- added CH1: SWD, $74th:2Pin, symbol $74th:SWD
- added CH3: WCH-Link-Header, $74th:WCH-Link-Port, symbol $74th:WCH-Link-Header
- C1: renamed from C2; footprint (none) -> $74th:Capacitor_0603_1608
- C2: renamed from C1; footprint (none) -> $74th:Capacitor_0603_1608
- C5: renamed from C3; value C -> 100n; footprint (none) -> $74th:Capacitor_0603_1608
- C6: footprint (none) -> $74th:Capacitor_0603_1608
- C7: renamed from C5; footprint (none) -> $74th:Capacitor_0603_1608
- C8: renamed from C4; footprint (none) -> $74th:Capacitor_0603_1608
- CH2: renamed from P1; value 1Pin -> RT; footprint (none) -> $74th:1Pin
- D1, D2: footprint (none) -> $74th:LED_0805_2012Metric_Pad1.15x1.40mm_HandSolder
- J1: footprint (none) -> $74th:USB-C-12-Pin-SMD
- R1: renamed from R2; footprint (none) -> $74th:Register_0603_1608
- R10: renamed from R9; footprint (none) -> $74th:Register_0603_1608
- R11: renamed from R10; footprint (none) -> $74th:Register_0603_1608
- R12: renamed from R11; footprint (none) -> $74th:Register_0603_1608
- R2: renamed from R3; footprint (none) -> $74th:Register_0603_1608
- R3: renamed from R7; footprint (none) -> $74th:Register_0603_1608
- R4: renamed from R8; footprint (none) -> $74th:Register_0603_1608
- R5: renamed from R6; footprint (none) -> $74th:Register_0603_1608
- R6: renamed from R5; footprint (none) -> $74th:Register_0603_1608
- R7: renamed from R4; footprint (none) -> $74th:Register_0603_1608
- R8: renamed from R1; footprint (none) -> $74th:Register_0603_1608
- R9: renamed from R12; footprint (none) -> $74th:Register_0603_1608
- U1: renamed from U3; footprint Package_TO_SOT_SMD:SOT-223-3_TabPin2 -> $74th:Regulator_AMS1117_SOT-89
- U2: renamed from U1; value ~ -> CH32V305FBP6; footprint (none) -> Package_SO:TSSOP-20_4.4x6.5mm_P0.65mm
- Y1: footprint (none) -> $74th:Crystal_SMD_3225-4Pin_3.2x2.5mm_HandSoldering
Connections:
- net +3V3: now also C3.2, CH3.7 (3V3)
- net +5V: now also C4.2, CH3.6 (5V)
- net D_SWCLK: now also CH1.1 (SWCLK)
- net D_SWDIO: now also CH1.2 (SWDIO)
- net GND: now also C3.1, C4.1, CH3.8 (GND)
- net RST: now also CH3.5 (RST)
- net at R1.2: now also CH3.10 (SWCLK)
- net at R3.1: now also CH3.1 (RX)
- net at R2.2: now also CH3.9 (SWDIO)
- net at R4.1: now also CH3.2 (TX)
- net at R5.1: now also CH3.3 (TDO)
- net at R6.1: now also CH3.4 (TDI)
Other:
- moved on the sheet: C5, D1, R1, R10, R2

Commit message: up
Parts:
- added CH4: IAP, $74th:1Pin, symbol $74th:1Pin
- Y1: value Oscillator_24GND -> 12M
Connections:
- net at R8.2, U2.10 (PC7): now also CH4.1
Changed lines of the file:
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@@
   (junction (at 96.52 102.87) (diameter 0) (color 0 0 0 0)
+  )
+  (junction (at 38.1 101.6) (diameter 0) (color 0 0 0 0)
   )
   (junction (at 204.47 43.18) (diameter 0) (color 0 0 0 0)
@@
   (symbol (lib_id "Device:R") (at 128.27 110.49 270) (unit 1)
     (in_bom yes) (on_board yes) (dnp no)
-    (property "Reference" "R1" (at 152.4 105.41 90)
+    (property "Reference" "R1" (at 128.27 105.41 90)
       (effects (font (size 1.27 1.27)))
     )
@@
         (path "/994bdb9a-227d-4e61-bdbf-a26950ab87e1"
           (reference "#PWR013") (unit 1)
+        )
+      )
+    )
+  )
+  (symbol (lib_id "$74th:1Pin") (at 31.75 101.6 0) (unit 1)
+    (in_bom yes) (on_board yes) (dnp no) (fields_autoplaced)
+    (property "Reference" "CH4" (at 31.75 96.52 0)
+      (effects (font (size 1.27 1.27)))
+    )
+    (property "Value" "IAP" (at 31.75 99.06 0)
+      (effects (font (size 1.27 1.27)))
+    )
+    (property "Footprint" "$74th:1Pin" (at 31.75 101.6 0)
+      (effects (font (size 1.27 1.27)) hide)
+    )
+    (property "Datasheet" "" (at 31.75 101.6 0)
+      (effects (font (size 1.27 1.27)) hide)
+    )
+    (pin "1")
+    (instances
+      (project "wch-link"
+        (path "/994bdb9a-227d-4e61-bdbf-a26950ab87e1"
+          (reference "CH4") (unit 1)
         )
       )
@@
       (effects (font (size 1.27 1.27)))
     )
-    (property "Value" "Oscillator_24GND" (at 133.35 56.7689 90)
-      (effects (font (size 1.27 1.27)))
-    )
+    (property "Value" "12M" (at 133.35 56.7689 90)
+      (effects (font (size 1.27 1.27)))
+    )

Commit message: v1.1.0
Parts:
- removed C6: 100n, $74th:Capacitor_0603_1608, symbol Device:C
- added J2: SWD-Debugger_Side-10Pin, $74th:BoxPinHeader_2x05_P1.27mm_Vertical, symbol $74th:SWD-Debugger_Side-10Pin
- added SW1: SW_Push, $74th:SKRPABE010, symbol Switch:SW_Push
- CH4: renamed from CH3; footprint $74th:WCH-Link-Port -> $74th:Side-2x5P-PinHeader-Right
- U1: footprint $74th:Regulator_AMS1117_SOT-89 -> Package_TO_SOT_SMD:SOT-223-3_TabPin2
- renumbered C3 to C2, C2 to C3, C7 to C6, C8 to C7, CH4 to CH1, CH1 to CH2, CH2 to CH3, R6 to R1, R8 to R10, R5 to R2, R1 to R5, R2 to R6, R9 to R8, R10 to R9
Connections:
- net +3V3: now also CH4.8 (3V3), J2.1 (VCC); no longer CH4.7 (3V3)
- net +5V: now also CH4.10 (5V); no longer CH4.6 (5V)
- net GND: now also CH4.6 (GND), J2.3 (GND), J2.5 (GND), J2.9 (GND), SW1.2; no longer CH4.8 (GND)
- net RST: now also CH4.9 (RST), J2.10 (~{RESET}); no longer CH4.5 (RST)
- net RX: now also CH4.1 (RX), J2.8 (RXD); no longer U2.4 (PB11)
- net TDI: now also CH4.7 (TDI); no longer U2.8 (PB15)
- net TDO: now also CH4.5 (TDO); no longer U2.7 (PB14)
- net TX: now also CH4.3 (TX), J2.7 (TXD); no longer U2.3 (PB10)
- net SWCLK/TCK: now reaches R5.2
- net SWCLK/TCK: now also CH4.2 (SWCLK), J2.4 (SWCLK); no longer CH4.10 (SWCLK)
- net at R3.1: now also U2.4 (PB11); no longer CH4.1 (RX)
- net ModeS: now reaches C1.2, U2.19 (OSC_IN/PD0), Y1.3
- net ModeS: now also SW1.1
- net at R4.1: now also U2.3 (PB10); no longer CH4.2 (TX)
- net at R2.1: now also U2.7 (PB14); no longer CH4.3 (TDO)
- net at R1.1: now also U2.8 (PB15); no longer CH4.4 (TDI)
- net SWDIO/TMS: now reaches R6.2
- net SWDIO/TMS: now also CH4.4 (SWDIO), J2.2 (SWDIO); no longer CH4.9 (SWDIO)
- net USB_N renamed USBD-
- net USB_P renamed USBD+
Other:
- moved on the sheet: C6, C7, CH1, D2, R1, R10, R2, R3, R4, R5, R6, R7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

Commit message: v1.1.0
Parts:
- D1: value LED -> BLUE
- D2: value LED -> RED
- R8: value 200 -> 1k
- R9: value 1k -> 10k
Changed lines of the file:
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@@
+    (stroke (width 0) (type default))
+  )
+  (wire (pts (xy 95.25 86.36) (xy 109.22 86.36))
     (stroke (width 0) (type default))
   )
@@
     (effects (font (size 1.27 1.27)) (justify right bottom))
   )
+  (label "RST" (at 109.22 86.36 180) (fields_autoplaced)
+    (effects (font (size 1.27 1.27)) (justify right bottom))
+  )
   (label "ModeS" (at 109.22 66.04 180) (fields_autoplaced)
     (effects (font (size 1.27 1.27)) (justify right bottom))
@@
     (effects (font (size 1.27 1.27)) (justify right bottom))
   )
-  (global_label "RST" (shape input) (at 95.25 86.36 0) (fields_autoplaced)
-    (effects (font (size 1.27 1.27)) (justify left))
-    (property "Intersheetrefs" "${INTERSHEET_REFS}" (at 101.6029 86.36 0)
-      (effects (font (size 1.27 1.27)) (justify left) hide)
-    )
-  )
   (symbol (lib_id "$74th:1Pin") (at 67.31 146.05 0) (unit 1)
     (in_bom yes) (on_board yes) (dnp no) (fields_autoplaced)
@@
   (symbol (lib_id "Device:R") (at 250.19 54.61 0) (unit 1)
     (in_bom yes) (on_board yes) (dnp no) (fields_autoplaced)
-    (property "Reference" "R8" (at 252.73 53.975 0)
+    (property "Reference" "R8" (at 252.73 53.34 0)
       (effects (font (size 1.27 1.27)) (justify left))
     )
-    (property "Value" "200" (at 252.73 56.515 0)
+    (property "Value" "1k" (at 252.73 55.88 0)
       (effects (font (size 1.27 1.27)) (justify left))
     )
@@
   (symbol (lib_id "Device:LED") (at 250.19 46.99 90) (unit 1)
     (in_bom yes) (on_board yes) (dnp no) (fields_autoplaced)
-    (property "Reference" "D2" (at 254 47.9425 90)
+    (property "Reference" "D2" (at 254 47.3075 90)
       (effects (font (size 1.27 1.27)) (justify right))
     )
-    (property "Value" "LED" (at 254 50.4825 90)
+    (property "Value" "RED" (at 254 49.8475 90)
       (effects (font (size 1.27 1.27)) (justify right))
     )
@@
   (symbol (lib_id "Device:R") (at 140.97 97.79 180) (unit 1)
     (in_bom yes) (on_board yes) (dnp no) (fields_autoplaced)
-    (property "Reference" "R9" (at 143.51 97.155 0)
+    (property "Reference" "R9" (at 143.51 96.52 0)
       (effects (font (size 1.27 1.27)) (justify right))
     )
-    (property "Value" "1k" (at 143.51 99.695 0)
+    (property "Value" "10k" (at 143.51 99.06 0)
       (effects (font (size 1.27 1.27)) (justify right))
     )
@@
   (symbol (lib_id "Device:LED") (at 140.97 90.17 90) (unit 1)
     (in_bom yes) (on_board yes) (dnp no) (fields_autoplaced)
-    (property "Reference" "D1" (at 144.78 91.1225 90)
+    (property "Reference" "D1" (at 144.78 90.4875 90)
       (effects (font (size 1.27 1.27)) (justify right))
     )
-    (property "Value" "LED" (at 144.78 93.6625 90)
+    (property "Value" "BLUE" (at 144.78 93.0275 90)
       (effects (font (size 1.27 1.27)) (justify right))
     )

Commit message: v1.1.1
Connections:
- net ModeS: now also C3.2, U2.20 (OSC_OUT/PD1), Y1.1; no longer C1.2, U2.19 (OSC_IN/PD0), Y1.3
- net IAP: now reaches CH1.1, R10.2, U2.10 (PC7)
- new net: C1.2, U2.19 (OSC_IN/PD0), Y1.3
Other:
- note added: "DAPLink Switch"
- note added: "Debugger SWD"
- note added: "MCU"
- note added: "POWER-USB"
- note added: "PinHeader"
- note added: "SWD BoxHeader"
- moved on the sheet: C1, C2, C3, C4, C5, C6, C7, CH1, CH2, CH3, CH4, D1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

Commit message: update docuemnts
Parts:
- J1: value USB2.0_C_v3 -> USB
Other:
- company: (none) -> 74th
- title: (none) -> WCH-LinkE Clone - Mini WCH LinkE
Changed lines of the file:
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@@
 (kicad_sch (version 20230121) (generator eeschema)
   (paper "A4")
+  (title_block
+    (title "WCH-LinkE Clone - Mini WCH LinkE")
+    (rev "1.1.1")
+    (company "74th")
+  )
   (junction (at 77.47 38.1) (diameter 0) (color 0 0 0 0)
   )
@@
   (symbol (lib_id "$74th:USB2.0_C_v3") (at 185.42 44.45 0) (unit 1)
     (in_bom yes) (on_board yes) (dnp no) (fields_autoplaced)
-    (property "Reference" "J1" (at 185.42 22.86 0)
-      (effects (font (size 1.27 1.27)))
-    )
-    (property "Value" "USB2.0_C_v3" (at 185.42 25.4 0)
-      (effects (font (size 1.27 1.27)))
-    )
+    (property "Reference" "J1" (at 185.42 21.59 0)
+      (effects (font (size 1.27 1.27)))
+    )
+    (property "Value" "USB" (at 185.42 24.13 0)
+      (effects (font (size 1.27 1.27)))
+    )
